File: Individual Board Projects/moduleBoard/ModuleBoard/ModuleBoard.kicad_sch (KiCad schematic)
At the start: 20 parts, among them IC1 MSPM0C1103SDGS20R, J1 Rotation Servo, J2 Extention Servo, J3 Debug, J4 5x2.54mm+2xBus, J5 5x2.54mm+2xBus, J6 5x2.54mm+2xBus, J7 5x2.54mm+2xBus, J8 5x2.54mm+2xBus, J9 5x2.54mm+2xBus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

Commit message: Module Layout Rev 0
Parts:
- SW1, SW2: footprint (none) -> Rose Actuator Library:button
Connections:
- net +3.3V: no longer C4.2, U1.3 (VDD)
- net +5V: now also C4.2, U1.3 (VDD)
- net nShoutIn1: now also IC1.3 (PA28_/_A5); no longer IC1.17 (PA22_/_A4)
- net nShoutIn2: now also IC1.17 (PA22_/_A4); no longer IC1.18 (PA23)
- net nShoutIn6: now also IC1.18 (PA23); no longer IC1.3 (PA28_/_A5)
- net Extention Bottom Out: now reaches IC1.11 (PA11), R2.1, SW1.1 (A), SW1.2 (A)
- net Rotation Key: now reaches IC1.12 (PA16_/_A8), R3.1, SW2.1 (A), SW2.2 (A)
Other:
- moved on the sheet: R3, SW2
Changed lines of the file:
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@@
 	)
 	(junction
-		(at 148.59 99.06)
+		(at 148.59 102.87)
 		(diameter 0)
 		(color 0 0 0 0)
@@
 	(wire
 		(pts
+			(xy 148.59 88.9) (xy 148.59 102.87)
+		)
+		(stroke
+			(width 0)
+			(type default)
+		)
+	)
+	(wire
+		(pts
 			(xy 44.45 57.15) (xy 44.45 58.42)
 		)
@@
 	(wire
 		(pts
-			(xy 148.59 88.9) (xy 148.59 99.06)
-		)
-		(stroke
-			(width 0)
-			(type default)
-		)
-	)
-	(wire
-		(pts
 			(xy 29.21 148.59) (xy 29.21 160.02)
 		)
@@
 	(wire
 		(pts
-			(xy 156.21 99.06) (xy 148.59 99.06)
+			(xy 154.94 102.87) (xy 148.59 102.87)
 		)
 		(stroke
@@
 	(wire
 		(pts
-			(xy 171.45 95.25) (xy 171.45 99.06)
+			(xy 171.45 95.25) (xy 171.45 102.87)
 		)
 		(stroke
@@
 	(wire
 		(pts
-			(xy 148.59 99.06) (xy 148.59 100.33)
+			(xy 148.59 102.87) (xy 148.59 104.14)
 		)
 		(stroke
@@
 	(wire
 		(pts
-			(xy 171.45 99.06) (xy 166.37 99.06)
+			(xy 171.45 102.87) (xy 165.1 102.87)
 		)
 		(stroke
@@
 	(wire
 		(pts
-			(xy 148.59 107.95) (xy 148.59 109.22)
+			(xy 148.59 111.76) (xy 148.59 113.03)
 		)
 		(stroke
@@
 		)
 	)
+	(label "Extention Bottom Out"
+		(at 143.51 115.57 90)
+		(effects
+			(font
+				(size 1.27 1.27)
+			)
+			(justify left bottom)
+		)
+	)
 	(label "Rotary Motor PWM"
 		(at 62.23 110.49 0)
@@
 		)
 	)
+	(label "Rotation Key"
+		(at 148.59 101.6 90)
+		(effects
+			(font
+				(size 1.27 1.27)
+			)
+			(justify left bottom)
+		)
+	)
 	(label "SWDIO"
 		(at 135.89 29.21 0)
@@
 		)
 	)
-	(hierarchical_label "nShoutIn6"
-		(shape input)
-		(at 83.82 73.66 180)
-		(effects
-			(font
-				(size 1.27 1.27)
-			)
-			(justify right)
-		)
-	)
 	(hierarchical_label "GND"
 		(shape bidirectional)
@@
 		)
 	)
+	(hierarchical_label "nShoutIn2"
+		(shape input)
+		(at 149.86 76.2 0)
+		(effects
+			(font
+				(size 1.27 1.27)
+			)
+			(justify left)
+		)
+	)
 	(hierarchical_label "nShoutIn4"
 		(shape output)
@@
 		)
 	)
+	(hierarchical_label "nShoutIn1"
+		(shape input)
+		(at 83.82 73.66 180)
+		(effects
+			(font
+				(size 1.27 1.27)
+			)
+			(justify right)
+		)
+	)
 	(hierarchical_label "GND"
 		(shape bidirectional)
@@
 		)
 	)
-	(hierarchical_label "nShoutIn2"
+	(hierarchical_label "nShoutIn6"
 		(shape input)
 		(at 149.86 73.66 0)
@@
 		)
 	)
-	(hierarchical_label "nShoutIn1"
-		(shape input)
-		(at 149.86 76.2 0)
-		(effects
-			(font
-				(size 1.27 1.27)
-			)
-			(justify left)
-		)
-	)
 	(hierarchical_label "GND"
 		(shape bidirectional)
@@
 	)
 	(symbol
+		(lib_id "power:+5V")
+		(at 87.63 26.67 0)
+		(unit 1)
+		(exclude_from_sim no)
+		(in_bom yes)
+		(on_board yes)
+		(dnp no)
+		(fields_autoplaced yes)
+		(property "Reference" "#PWR01"
+			(at 87.63 30.48 0)
+			(effects
+				(font
+					(size 1.27 1.27)
+				)
+				(hide yes)
+			)
+		)
+		(property "Value" "+5V"
+			(at 87.63 21.59 0)
+			(effects
+				(font
+					(size 1.27 1.27)
+				)
+			)
+		)
+		(property "Footprint" ""
+			(at 87.63 26.67 0)
+			(effects
+				(font
+					(size 1.27 1.27)
+				)
+				(hide yes)
+			)
+		)
+		(property "Datasheet" ""
+			(at 87.63 26.67 0)
+			(effects
+				(font
+					(size 1.27 1.27)
+				)
+				(hide yes)
+			)
+		)
+		(property "Description" "Power symbol creates a global label with name \"+5V\""
+			(at 87.63 26.67 0)
+			(effects
+				(font
+					(size 1.27 1.27)
+				)
+				(hide yes)
+			)
+		)
+		(pin "1"
+		)
+		(instances
+			(project "ModuleBoard"
+				(path "/87dd8ead-887e-465a-b455-9f6b34d0a10e"
+					(reference "#PWR01")
+					(unit 1)
+				)
+			)
+		)
+	)
+	(symbol
 		(lib_id "Connector_Generic:Conn_01x07")
 		(at 208.28 40.64 0)
@@
 	(symbol
 		(lib_id "power:GND")
-		(at 148.59 109.22 0)
+		(at 148.59 113.03 0)
 		(unit 1)
 		(exclude_from_sim no)
@@
 		(fields_autoplaced yes)
 		(property "Reference" "#PWR0109"
-			(at 148.59 115.57 0)
+			(at 148.59 119.38 0)
 			(effects
 				(font
@@
 		)
 		(property "Value" "GND"
-			(at 148.59 114.3 0)
+			(at 148.59 118.11 0)
 			(effects
 				(font
@@
 		)
 		(property "Footprint" ""
-			(at 148.59 109.22 0)
+			(at 148.59 113.03 0)
 			(effects
 				(font
@@
 		)
 		(property "Datasheet" ""
-			(at 148.59 109.22 0)
+			(at 148.59 113.03 0)
 			(effects
 				(font
@@
 		)
 		(property "Description" "Power symbol creates a global label with name \"GND\" , ground"
-			(at 148.59 109.22 0)
+			(at 148.59 113.03 0)
 			(effects
 				(font
@@
 	)
 	(symbol
-		(lib_id "power:+3.3V")
-		(at 87.63 26.67 0)
-		(unit 1)
-		(exclude_from_sim no)
-		(in_bom yes)
-		(on_board yes)
-		(dnp no)
-		(fields_autoplaced yes)
-		(property "Reference" "#PWR0116"
-			(at 87.63 30.48 0)
-			(effects
-				(font
-					(size 1.27 1.27)
-				)
-				(hide yes)
-			)
-		)
-		(property "Value" "+3.3V"
-			(at 87.63 21.59 0)
-			(effects
-				(font
-					(size 1.27 1.27)
-				)
-			)
-		)
-		(property "Footprint" ""
-			(at 87.63 26.67 0)
-			(effects
-				(font
-					(size 1.27 1.27)
-				)
-				(hide yes)
-			)
-		)
-		(property "Datasheet" ""
-			(at 87.63 26.67 0)
-			(effects
-				(font
-					(size 1.27 1.27)
-				)
-				(hide yes)
-			)
-		)
-		(property "Description" "Power symbol creates a global label with name \"+3.3V\""
-			(at 87.63 26.67 0)
-			(effects
-				(font
-					(size 1.27 1.27)
-				)
-				(hide yes)
-			)
-		)
-		(pin "1"
-		)
-		(instances
-			(project "ModuleBoard"
-				(path "/87dd8ead-887e-465a-b455-9f6b34d0a10e"
-					(reference "#PWR0116")
-					(unit 1)
-				)
-			)
-		)
-	)
-	(symbol
 		(lib_id "Connector_Generic:Conn_01x07")
 		(at 208.28 91.44 0)
@@
 			)
 		)
-		(property "Footprint" ""
+		(property "Footprint" "Rose Actuator Library:button"
 			(at 154.94 116.84 0)
 			(effects
@@
 	(symbol
 		(lib_id "Device:R_US")
-		(at 148.59 104.14 0)
+		(at 148.59 107.95 0)
 		(unit 1)
 		(exclude_from_sim no)
@@
 		(fields_autoplaced yes)
 		(property "Reference" "R3"
-			(at 151.13 102.8699 0)
+			(at 151.13 106.6799 0)
 			(effects
 				(font
@@
 		)
 		(property "Value" "40k"
-			(at 151.13 105.4099 0)
+			(at 151.13 109.2199 0)
 			(effects
 				(font
@@
 		)
 		(property "Footprint" "Resistor_SMD:R_1206_3216Metric_Pad1.30x1.75mm_HandSolder"
-			(at 149.606 104.394 90)
+			(at 149.606 108.204 90)
 			(effects
 				(font
@@
 		)
 		(property "Datasheet" "~"
-			(at 148.59 104.14 0)
+			(at 148.59 107.95 0)
 			(effects
 				(font
@@
 		)
 		(property "Description" "Resistor, US symbol"
-			(at 148.59 104.14 0)
+			(at 148.59 107.95 0)
 			(effects
 				(font
@@
 	(symbol
 		(lib_id "Switch:SW_MEC_5G")
-		(at 161.29 99.06 0)
+		(at 160.02 102.87 0)
 		(unit 1)
 		(exclude_from_sim no)
@@
 		(fields_autoplaced yes)
 		(property "Reference" "SW2"
-			(at 161.29 91.44 0)
+			(at 160.02 95.25 0)
 			(effects
 				(font
@@
 		)
 		(property "Value" "SW_MEC_5G"
-			(at 161.29 93.98 0)
+			(at 160.02 97.79 0)
 			(effects
 				(font
@@
 			)
 		)
-		(property "Footprint" ""
-			(at 161.29 93.98 0)
+		(property "Footprint" "Rose Actuator Library:button"
+			(at 160.02 97.79 0)
 			(effects
 				(font
@@
 		)
 		(property "Datasheet" "http://www.apem.com/int/index.php?controller=attachment&id_attachment=488"
-			(at 161.29 93.98 0)
+			(at 160.02 97.79 0)
 			(effects
 				(font
@@
 		)
 		(property "Description" "MEC 5G single pole normally-open tactile switch"
-			(at 161.29 99.06 0)
+			(at 160.02 102.87 0)
 			(effects
 				(font
