File: Individual Board Projects/interConnectBoard/InterConnect/InterConnect.kicad_sch (KiCad schematic)
At the start: 2 parts, among them J1 5x2.54mm+2xBus, J2 5x2.54mm+2xBus

Commit message: Interconnect Board
Parts:
- J1, J2: footprint (none) -> Rose Actuator Library:InterconecsIside
Changed lines of the file:
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@@
 			)
 		)
-		(property "Footprint" ""
+		(property "Footprint" "Rose Actuator Library:InterconecsIside"
 			(at 124.46 100.33 0)
 			(effects
@@
 			)
 		)
-		(property "Footprint" ""
+		(property "Footprint" "Rose Actuator Library:InterconecsIside"
 			(at 167.64 100.33 0)
 			(effects
