File: Individual Board Projects/controlBoard/ControlBoard/ControlBoard.kicad_sch (KiCad schematic)
At the start: 12 parts, among them J1 USBCPD, J2 AudioJack3, J3 5x2.54mm+2xBus, U1 LMC6484, U2 LMC6484, U3 ESP32-C6-DEVKITC-1-N8

Commit message: Updated KiCad files
Parts:
- removed J2: AudioJack3, symbol Connector_Audio:AudioJack3
- removed U1, U2: LMC6484, Rose Actuator Library:DIP254P762X508-14, symbol Amplifier_Operational:LMC6484
- added J4: MJ1-2503A, Rose Actuator Library:SAMESKY_MJ1-2503A, symbol Rosethings:MJ1-2503A
- added U1: LMC6484IN_NOPB, Rose Actuator Library:DIP254P762X508-14, symbol LMC6484IN_NOPB:LMC6484IN_NOPB
- added U2: 01000020Z, 01000020Z, symbol Rosethings:01000020Z
- B1: footprint (none) -> BUCK_and_USBC:Buck-fourpins
- J1: footprint (none) -> BUCK_and_USBC:USBC-PD-Module-twopins
Connections:
- net +1.65V: now also J4.1
- net +3.3V: now also U1.4 (V+)
- net GND: now also U1.11 (V-)
- net To ESP32 ADC: now also U1.1 (OUT1)
- net at R3.1, RV1.1: now also U1.2 (NEG1)
- new net: J4.3, U1.3 (POS1)
- no-connect marks 22 -> 21
Other:
- moved on the sheet: R3, RV1

Commit message: Updated ControlBoard design files
Parts:
- RV1: footprint (none) -> BUCK_and_USBC:Potentiometer
- U2: footprint 01000020Z -> BUCK_and_USBC:01000020Z
Connections:
- net +5V: now also U2.2; no longer B1.3 (+Vout)
- net at U2.1: now also B1.3 (+Vout)
Other:
- moved on the sheet: U2
Changed lines of the file:
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@@
 	(wire
 		(pts
+			(xy 39.37 49.53) (xy 54.61 49.53)
+		)
+		(stroke
+			(width 0)
+			(type default)
+		)
+	)
+	(wire
+		(pts
 			(xy 243.84 102.87) (xy 254 102.87)
 		)
@@
 	(wire
 		(pts
+			(xy 96.52 45.72) (xy 100.33 45.72)
+		)
+		(stroke
+			(width 0)
+			(type default)
+		)
+	)
+	(wire
+		(pts
 			(xy 113.03 105.41) (xy 113.03 107.95)
 		)
@@
 	(wire
 		(pts
-			(xy 58.42 80.01) (xy 67.31 80.01)
+			(xy 100.33 57.15) (xy 107.95 57.15)
 		)
 		(stroke
@@
 	(wire
 		(pts
-			(xy 177.8 100.33) (xy 195.58 100.33)
+			(xy 58.42 80.01) (xy 67.31 80.01)
 		)
 		(stroke
@@
 	(wire
 		(pts
-			(xy 177.8 107.95) (xy 195.58 107.95)
+			(xy 177.8 100.33) (xy 195.58 100.33)
 		)
 		(stroke
@@
 	(wire
 		(pts
-			(xy 177.8 74.93) (xy 195.58 74.93)
+			(xy 177.8 107.95) (xy 195.58 107.95)
 		)
 		(stroke
@@
 	(wire
 		(pts
-			(xy 132.08 96.52) (xy 132.08 100.33)
+			(xy 177.8 74.93) (xy 195.58 74.93)
 		)
 		(stroke
@@
 	(wire
 		(pts
-			(xy 93.98 49.53) (xy 90.17 49.53)
+			(xy 132.08 96.52) (xy 132.08 100.33)
 		)
 		(stroke
@@
 	(wire
 		(pts
+			(xy 90.17 49.53) (xy 96.52 49.53)
+		)
+		(stroke
+			(width 0)
+			(type default)
+		)
+	)
+	(wire
+		(pts
 			(xy 234.95 95.25) (xy 254 95.25)
 		)
@@
 	(wire
 		(pts
-			(xy 54.61 49.53) (xy 39.37 49.53)
+			(xy 121.92 72.39) (xy 121.92 67.31)
 		)
 		(stroke
@@
 	(wire
 		(pts
-			(xy 121.92 72.39) (xy 121.92 67.31)
+			(xy 177.8 80.01) (xy 195.58 80.01)
 		)
 		(stroke
@@
 	(wire
 		(pts
-			(xy 177.8 80.01) (xy 195.58 80.01)
+			(xy 105.41 96.52) (xy 105.41 101.6)
 		)
 		(stroke
@@
 	(wire
 		(pts
-			(xy 105.41 96.52) (xy 105.41 101.6)
+			(xy 41.91 123.19) (xy 41.91 127)
 		)
 		(stroke
@@
 	(wire
 		(pts
-			(xy 41.91 123.19) (xy 41.91 127)
+			(xy 100.33 48.26) (xy 100.33 57.15)
 		)
 		(stroke
@@
 	(wire
 		(pts
+			(xy 96.52 49.53) (xy 96.52 45.72)
+		)
+		(stroke
+			(width 0)
+			(type default)
+		)
+	)
+	(wire
+		(pts
 			(xy 105.41 90.17) (xy 105.41 96.52)
 		)
@@
 	(symbol
 		(lib_id "power:+5V")
-		(at 93.98 49.53 0)
+		(at 107.95 57.15 0)
 		(unit 1)
 		(exclude_from_sim no)
@@
 		(fields_autoplaced yes)
 		(property "Reference" "#PWR0109"
-			(at 93.98 53.34 0)
+			(at 107.95 60.96 0)
 			(effects
 				(font
@@
 		)
 		(property "Value" "+5V"
-			(at 93.98 44.45 0)
+			(at 107.95 52.07 0)
 			(effects
 				(font
@@
 		)
 		(property "Footprint" ""
-			(at 93.98 49.53 0)
+			(at 107.95 57.15 0)
 			(effects
 				(font
@@
 		)
 		(property "Datasheet" ""
-			(at 93.98 49.53 0)
+			(at 107.95 57.15 0)
 			(effects
 				(font
@@
 		)
 		(property "Description" "Power symbol creates a global label with name \"+5V\""
-			(at 93.98 49.53 0)
+			(at 107.95 57.15 0)
 			(effects
 				(font
@@
 			)
 		)
-		(property "Footprint" ""
+		(property "Footprint" "BUCK_and_USBC:Potentiometer"
 			(at 105.41 105.41 0)
 			(effects
@@
 	(symbol
 		(lib_id "Rosethings:01000020Z")
-		(at 91.44 71.12 0)
+		(at 100.33 45.72 0)
 		(unit 1)
 		(exclude_from_sim no)
@@
 		(fields_autoplaced yes)
 		(property "Reference" "U2"
-			(at 107.95 71.1199 0)
+			(at 116.84 45.7199 0)
 			(effects
 				(font
@@
 		)
 		(property "Value" "01000020Z"
-			(at 107.95 73.6599 0)
+			(at 116.84 48.2599 0)
 			(effects
 				(font
@@
 			)
 		)
-		(property "Footprint" "01000020Z"
-			(at 107.95 166.04 0)
+		(property "Footprint" "BUCK_and_USBC:01000020Z"
+			(at 116.84 140.64 0)
 			(effects
 				(font
@@
 		)
 		(property "Datasheet" "https://componentsearchengine.com/Datasheets/1/01000020Z.pdf"
-			(at 107.95 266.04 0)
+			(at 116.84 240.64 0)
 			(effects
 				(font
@@
 		)
 		(property "Description" "Littelfuse Fuse Holder Clip"
-			(at 91.44 71.12 0)
+			(at 100.33 45.72 0)
 			(effects
 				(font
@@
 		)
 		(property "Height" "10.7"
-			(at 107.95 466.04 0)
+			(at 116.84 440.64 0)
 			(effects
 				(font
@@
 		)
 		(property "Mouser Part Number" "576-01000020Z"
-			(at 107.95 566.04 0)
+			(at 116.84 540.64 0)
 			(effects
 				(font
@@
 		)
 		(property "Mouser Price/Stock" "https://www.mouser.co.uk/ProductDetail/Littelfuse/01000020Z?qs=A2K%252BDn3pTTkC2o2QQivHQg%3D%3D"
-			(at 107.95 666.04 0)
+			(at 116.84 640.64 0)
 			(effects
 				(font
@@
 		)
 		(property "Manufacturer_Name" "LITTELFUSE"
-			(at 107.95 766.04 0)
+			(at 116.84 740.64 0)
 			(effects
 				(font
@@
 		)
 		(property "Manufacturer_Part_Number" "01000020Z"
-			(at 107.95 866.04 0)
+			(at 116.84 840.64 0)
 			(effects
 				(font
